Commit message: added ros2 control code

File: ros2_ws/src/low_cost_robot_description/urdf/low_cost_robot.xacro (robot description, xacro)
@@ -2,6 +2,7 @@
 <robot name="low_cost_robot" xmlns:xacro="http://www.ros.org/wiki/xacro">
 <xacro:include filename="$(find low_cost_robot_description)/urdf/materials.xacro" />
-<xacro:include filename="$(find low_cost_robot_description)/urdf/low_cost_robot.trans" />
-<xacro:include filename="$(find low_cost_robot_description)/urdf/low_cost_robot.gazebo" />
+<!-- <xacro:include filename="$(find low_cost_robot_description)/urdf/low_cost_robot.trans" /> -->
+<!-- <xacro:include filename="$(find low_cost_robot_description)/urdf/low_cost_robot.gazebo" /> -->
+<xacro:include filename="$(find low_cost_robot_description)/urdf/ros2_control.xacro" />
 <link name="base_link">
   <inertial>
@@ -24,4 +25,7 @@
   </collision>
 </link>
+<gazebo reference="base_link">
+  <material>Gazebo/Red</material>
+</gazebo>
 <link name="link1_1">
   <inertial>
@@ -44,4 +48,7 @@
   </collision>
 </link>
+<gazebo reference="link1_1">
+  <material>Gazebo/Green</material>
+</gazebo>
 <link name="link2_1">
   <inertial>
@@ -64,4 +71,7 @@
   </collision>
 </link>
+<gazebo reference="link2_1">
+  <material>Gazebo/Blue</material>
+</gazebo>
 <link name="link3_1">
   <inertial>
@@ -84,4 +94,7 @@
   </collision>
 </link>
+<gazebo reference="link3_1">
+  <material>Gazebo/Yellow</material>
+</gazebo>
 <link name="link4_1">
   <inertial>
@@ -104,4 +117,7 @@
   </collision>
 </link>
+<gazebo reference="link4_1">
+  <material>Gazebo/Orange</material>
+</gazebo>
 <link name="gripper_static_1">
   <inertial>
@@ -124,4 +140,7 @@
   </collision>
 </link>
+<gazebo reference="gripper_static_1">
+  <material>Gazebo/Purple</material>
+</gazebo>
 <link name="gripper_moving_1">
   <inertial>
@@ -144,4 +163,7 @@
   </collision>
 </link>
+<gazebo reference="gripper_moving_1">
+  <material>Gazebo/Turquoise</material>
+</gazebo>
 <joint name="joint1" type="continuous">
   <origin xyz="0.0 0.0 0.039" rpy="0 0 0"/>
